Commit message: fix bno08x and base_footprint

File: diffdrive_real_hw/description/urdf/robot.urdf.xacro (robot description, xacro)
@@ -4,10 +4,13 @@
   <!--  Parameters  — edit to match your robot                           -->
   <!-- ================================================================ -->
-  <xacro:property name="base_length"      value="0.200"/>
-  <xacro:property name="base_width"       value="0.180"/>
-  <xacro:property name="base_height"      value="0.080"/>
+  <xacro:property name="base_length"      value="0.400"/>
+  <xacro:property name="base_width"       value="0.350"/>
+  <xacro:property name="base_height"      value="0.10"/>
   <xacro:property name="wheel_radius"     value="0.033"/>
   <xacro:property name="wheel_thickness"  value="0.020"/>
-  <xacro:property name="wheel_separation" value="0.160"/>
+  <xacro:property name="wheel_separation" value="0.310"/>
+  <!-- Sensor offsets -->
+  <xacro:property name="lidar_height"     value="0.01"/>  <!-- LiDAR body half-height -->
+  <xacro:property name="imu_size"         value="0.025"/>  <!-- IMU box side length -->
   <!-- ================================================================ -->
   <!--  Links & Joints                                                    -->
@@ -17,5 +20,5 @@
     <parent link="base_footprint"/>
     <child  link="base_link"/>
-    <origin xyz="0 0 ${wheel_radius}" rpy="0 0 0"/>
+    <origin xyz="0 0 ${wheel_radius + 0.04}" rpy="0 0 0"/>
   </joint>
   <link name="base_link">
@@ -51,5 +54,5 @@
       <parent link="base_link"/>
       <child  link="${name}"/>
-      <origin xyz="0 ${y_reflect * wheel_separation / 2} 0" rpy="0 0 0"/>
+      <origin xyz="0 ${y_reflect * wheel_separation / 2} -0.04" rpy="0 0 0"/>
       <axis xyz="0 1 0"/>
     </joint>
@@ -75,22 +78,63 @@
   </joint>
   <!-- ================================================================ -->
+  <!--  IMU                                                               -->
+  <!--  Centered on top of base. Frame aligned with base_link (no rpy). -->
+  <!--  Edit xyz to match your physical mounting position.               -->
+  <!-- ================================================================ -->
+  <link name="imu_link">
+    <visual>
+      <geometry><box size="${imu_size} ${imu_size} 0.010"/></geometry>
+      <material name="green"><color rgba="0.0 0.8 0.2 1.0"/></material>
+    </visual>
+    <collision>
+      <geometry><box size="${imu_size} ${imu_size} 0.010"/></geometry>
+    </collision>
+    <inertial>
+      <mass value="0.010"/>
+      <inertia ixx="0.000001" ixy="0" ixz="0" iyy="0.000001" iyz="0" izz="0.000001"/>
+    </inertial>
+  </link>
+  <joint name="imu_joint" type="fixed">
+    <parent link="base_link"/>
+    <child  link="imu_link"/>
+    <!-- Sits on top of the base, centered -->
+    <origin xyz="0 0 0.005" rpy="0 0 0"/>
+  </joint>
+  <!-- ================================================================ -->
+  <!--  LiDAR                                                             -->
+  <!--  Mounted forward-center on top of base. Adjust xyz as needed.    -->
+  <!--  The laser scan plane is at z=0 of lidar_link by convention.     -->
+  <!-- ================================================================ -->
+  <link name="lidar_link">
+    <visual>
+      <geometry><cylinder radius="0.035" length="${lidar_height * 2}"/></geometry>
+      <material name="black"><color rgba="0.1 0.1 0.1 1.0"/></material>
+    </visual>
+    <collision>
+      <geometry><cylinder radius="0.035" length="${lidar_height * 2}"/></geometry>
+    </collision>
+    <inertial>
+      <mass value="0.150"/>
+      <inertia ixx="0.0001" ixy="0" ixz="0" iyy="0.0001" iyz="0" izz="0.0001"/>
+    </inertial>
+  </link>
+  <joint name="lidar_joint" type="fixed">
+    <parent link="base_link"/>
+    <child  link="lidar_link"/>
+    <!-- Forward-center, scan plane level with top of lidar body -->
+    <origin xyz="0 0 ${base_height/2 + lidar_height}" rpy="0 0 0"/>
+  </joint>
+  <!-- ================================================================ -->
   <!--  ros2_control hardware interface block                             -->
-  <!--                                                                   -->
-  <!--  Plugin: esp32_hardware/Esp32HardwareInterface                    -->
-  <!--  Parameters are read by on_init() in the C++ plugin.              -->
-  <!--                                                                   -->
-  <!--  serial_port: your ESP32's USB serial device                      -->
-  <!--  baud_rate:   must match Serial.begin() in firmware               -->
   <!-- ================================================================ -->
   <ros2_control name="esp32_hardware" type="system">
     <hardware>
       <plugin>esp32_hardware/Esp32HardwareInterface</plugin>
-      <param name="serial_port">/dev/serial/by-id/usb-1a86_USB_Serial-if00-port0</param>   <!-- ← edit this -->
+      <param name="serial_port">/dev/serial/by-id/usb-1a86_USB_Serial-if00-port0</param>
       <param name="baud_rate">921600</param>
     </hardware>
-    <!-- Joint order: index 0 = left, 1 = right (matches ESP32 firmware) -->
     <joint name="left_wheel_joint">
       <command_interface name="velocity">
-        <param name="min">-9.0</param>   <!-- rad/s, matches MAX_VEL in firmware -->
+        <param name="min">-9.0</param>
         <param name="max"> 9.0</param>
       </command_interface>
